Commit message: camera + monza

File: install/my_robot_description/share/my_robot_description/urdf/mobile_base_gazebo.xacro (robot description, xacro)
@@ -1,4 +1,5 @@
 <?xml version="1.0"?>
 <robot xmlns:xacro="http://www.ros.org/wiki/xacro">
+    <xacro:property name="FOV" value="60" />
     <gazebo>
         <plugin filename="gz-sim-diff-drive-system" name="gz::sim::systems::DiffDrive">
@@ -21,3 +22,23 @@
         </plugin>
     </gazebo>
+    <gazebo reference="camera_link">
+        <sensor type="camera" name="drive_camera">
+            <pose relative_to='camera_link'>0 0 0 0 0 0</pose>
+            <camera>
+                <horizontal_fov>${FOV * pi / 180}</horizontal_fov>
+                <image>
+                <width>720</width>
+                <height>480</height>
+                </image>
+                <clip>
+                <near>0.1</near>
+                <far>100</far>
+                </clip>
+            </camera>
+            <always_on>1</always_on>
+            <update_rate>15</update_rate>
+            <visualize>true</visualize>
+            <topic>camera/image_raw</topic>
+        </sensor>
+    </gazebo>
 </robot>

File: install/my_robot_description/share/my_robot_description/urdf/my_robot.urdf.xacro (robot description, xacro)
@@ -6,4 +6,5 @@
     <xacro:property name="wheel_radius" value="0.1" />
     <xacro:property name="wheel_length" value="0.05" />
+    <xacro:property name="camera_side_length" value="0.04" />
     <xacro:include filename="$(find my_robot_description)/urdf/common_properties.xacro" />
     <xacro:include filename="$(find my_robot_description)/urdf/mobile_base_gazebo.xacro" />
@@ -14,4 +15,15 @@
         <color rgba="0.7 0.7 0.7 1" />
     </material>
+    <link name="camera_link">
+        <xacro:box_inertia m="0.01" x="${camera_side_length}" y="${camera_side_length}"
+        z="${camera_side_length}" o_xyz="${camera_side_length / 2} 0 0" o_rpy="0 0 0" />
+        <visual>
+            <geometry>
+                <box size="${camera_side_length} ${camera_side_length} ${camera_side_length}" />
+            </geometry>
+            <origin xyz="${camera_side_length / 2} 0 0" rpy="0 0 0" />
+            <material name="gray" />
+        </visual>
+    </link>
     <link name="base_link">
         <xacro:box_inertia m="5.0" x="${base_length}" y="${base_width}" z="${base_height}"
@@ -93,4 +105,9 @@
     </link>
     <link name="base_footprint" />
+    <joint name="base_camera_joint" type="fixed">
+        <parent link="base_link" />
+        <child link="camera_link" />
+        <origin xyz="${base_length / 2} 0 ${base_height}" rpy="0 0 0" />
+    </joint>
     <joint name="base_shoulder_joint" type="revolute">
         <parent link="base_link" />
@@ -104,5 +121,5 @@
         <child link="right_wheel_link" />
         <origin xyz="${-base_length / 4.0} ${-(base_width + wheel_length) /
-            2.0} 0" rpy="0 ${pi / 2.0} 0" />
+            2.0} 0" rpy="0 0 0" />
         <axis xyz="0 1 0" />
     </joint>
