Commit message: full terrain no NPC

File: install/my_robot_description/share/my_robot_description/urdf/common_properties.xacro (robot description, xacro)
@@ -1,33 +1 @@
-<?xml version="1.0"?>
-<robot xmlns:xacro="http://www.ros.org/wiki/xacro">
-    <!-- Box Inertia Macro -->
-    <xacro:macro name="box_inertia" params="m x y z o_xyz o_rpy">
-    <inertial>
-        <mass value="${m}" />
-        <origin xyz="${o_xyz}" rpy="${o_rpy}" />
-        <inertia ixx="${(m/12) * (y*y + z*z)}" ixy="0" ixz="0"
-                iyy="${(m/12) * (x*x + z*z)}" iyz="0"
-                izz="${(m/12) * (x*x + y*y)}" />
-    </inertial>
-    </xacro:macro>
-    <!-- Cylinder Inertia Macro -->
-    <xacro:macro name="cylinder_inertia" params="m r l o_xyz o_rpy">
-    <inertial>
-        <mass value="${m}" />
-        <origin xyz="${o_xyz}" rpy="${o_rpy}" />
-        <inertia ixx="${(m/12) * (3*r*r + l*l)}" ixy="0" ixz="0"
-                iyy="${(m/12) * (3*r*r + l*l)}" iyz="0"
-                izz="${(m/2) * (r*r)}" />
-    </inertial>
-    </xacro:macro>
-    <!-- Sphere Inertia Macro -->
-    <xacro:macro name="sphere_inertia" params="m r o_xyz o_rpy">
-    <inertial>
-        <mass value="${m}" />
-        <origin xyz="${o_xyz}" rpy="${o_rpy}" />
-        <inertia ixx="${(2/5) * m * r * r}" ixy="0" ixz="0"
-                iyy="${(2/5) * m * r * r}" iyz="0"
-                izz="${(2/5) * m * r * r}" />
-    </inertial>
-    </xacro:macro>
-</robot>
+/home/fizzer/my_robot_ws/src/my_robot_description/urdf/common_properties.xacro

File: install/my_robot_description/share/my_robot_description/urdf/mobile_base_gazebo.xacro (robot description, xacro)
@@ -1,44 +1 @@
-<?xml version="1.0"?>
-<robot xmlns:xacro="http://www.ros.org/wiki/xacro">
-    <xacro:property name="FOV" value="60" />
-    <gazebo>
-        <plugin filename="gz-sim-diff-drive-system" name="gz::sim::systems::DiffDrive">
-            <left_joint>base_left_wheel_joint</left_joint>
-            <right_joint>base_right_wheel_joint</right_joint>
-            <frame_id>odom</frame_id>
-            <child_frame_id>base_footprint</child_frame_id>
-            <wheel_separation>0.45</wheel_separation>
-            <wheel_radius>0.1</wheel_radius>
-        </plugin>
-    </gazebo>
-    <gazebo reference="caster_wheel_link">
-        <mu1 value="0.1" />
-        <mu2 value="0.1" />
-    </gazebo>
-    <gazebo>
-        <plugin
-            filename="gz-sim-joint-state-publisher-system"
-            name="gz::sim::systems::JointStatePublisher">
-        </plugin>
-    </gazebo>
-    <gazebo reference="camera_link">
-        <sensor type="camera" name="drive_camera">
-            <pose relative_to='camera_link'>0 0 0 0 0 0</pose>
-            <camera>
-                <horizontal_fov>${FOV * pi / 180}</horizontal_fov>
-                <image>
-                <width>720</width>
-                <height>480</height>
-                </image>
-                <clip>
-                <near>0.1</near>
-                <far>100</far>
-                </clip>
-            </camera>
-            <always_on>1</always_on>
-            <update_rate>15</update_rate>
-            <visualize>true</visualize>
-            <topic>camera/image_raw</topic>
-        </sensor>
-    </gazebo>
-</robot>
+/home/fizzer/my_robot_ws/src/my_robot_description/urdf/mobile_base_gazebo.xacro

File: install/my_robot_description/share/my_robot_description/urdf/my_robot.urdf.xacro (robot description, xacro)
@@ -1,143 +1 @@
-<?xml version="1.0"?>
-<robot name="my_robot" xmlns:xacro="http://www.ros.org/wiki/xacro">
-    <xacro:property name="base_length" value="0.6" />
-    <xacro:property name="base_width" value="0.4" />
-    <xacro:property name="base_height" value="0.2" />
-    <xacro:property name="wheel_radius" value="0.1" />
-    <xacro:property name="wheel_length" value="0.05" />
-    <xacro:property name="camera_side_length" value="0.04" />
-    <xacro:include filename="$(find my_robot_description)/urdf/common_properties.xacro" />
-    <xacro:include filename="$(find my_robot_description)/urdf/mobile_base_gazebo.xacro" />
-    <material name="green">
-        <color rgba="0 0.6 0 1" />
-    </material>
-    <material name="gray">
-        <color rgba="0.7 0.7 0.7 1" />
-    </material>
-    <link name="camera_link">
-        <xacro:box_inertia m="0.01" x="${camera_side_length}" y="${camera_side_length}"
-        z="${camera_side_length}" o_xyz="${camera_side_length / 2} 0 0" o_rpy="0 0 0" />
-        <visual>
-            <geometry>
-                <box size="${camera_side_length} ${camera_side_length} ${camera_side_length}" />
-            </geometry>
-            <origin xyz="${camera_side_length / 2} 0 0" rpy="0 0 0" />
-            <material name="gray" />
-        </visual>
-    </link>
-    <link name="base_link">
-        <xacro:box_inertia m="5.0" x="${base_length}" y="${base_width}" z="${base_height}"
-        o_xyz="0 0 ${base_height / 2.0}" o_rpy="0 0 0" />
-        <collision>
-            <origin xyz="0 0 ${base_height / 2.0}" rpy="0 0 0" />
-            <geometry>
-                <box size="${base_length} ${base_width} ${base_height}" />
-            </geometry>
-        </collision>
-        <visual>
-            <geometry>
-                <box size="${base_length} ${base_width} ${base_height}" />
-            </geometry>
-            <origin xyz="0 0 ${base_height / 2.0}" rpy="0 0 0" />
-            <material name="green" />
-        </visual>
-    </link>
-    <link name="shoulder_link">
-        <xacro:cylinder_inertia m="1.0" r="0.1" l="0.3"
-        o_xyz="0 0 0.15" o_rpy="0 0 0" />
-        <visual>
-            <geometry>
-                <cylinder radius="0.1" length="0.3" />
-            </geometry>
-            <origin xyz="0 0 0.15" rpy="0 0 0" />
-            <material name="gray" />
-        </visual>
-    </link>
-    <link name="right_wheel_link">
-        <xacro:cylinder_inertia m="1.0" r="${wheel_radius}" l="${wheel_length}"
-        o_xyz="0 0 0" o_rpy="${pi / 2.0} 0 0" />
-        <collision>
-            <origin xyz="0 0 0" rpy="0 0 0" />
-            <geometry>
-                <sphere radius="${wheel_radius}" />
-            </geometry>
-        </collision>
-        <visual>
-            <geometry>
-                <cylinder radius="${wheel_radius}" length="${wheel_length}" />
-            </geometry>
-            <origin xyz="0 0 0" rpy="${pi / 2.0} 0 0" />
-            <material name="gray" />
-        </visual>
-    </link>
-    <link name="left_wheel_link">
-        <xacro:cylinder_inertia m="1.0" r="${wheel_radius}" l="${wheel_length}"
-        o_xyz="0 0 0" o_rpy="${pi / 2.0} 0 0" />
-        <collision>
-            <origin xyz="0 0 0" rpy="0 0 0" />
-            <geometry>
-                <sphere radius="${wheel_radius}" />
-            </geometry>
-        </collision>
-        <visual>
-            <geometry>
-                <cylinder radius="${wheel_radius}" length="${wheel_length}" />
-            </geometry>
-            <origin xyz="0 0 0" rpy="${-pi / 2.0} 0 0" />
-            <material name="gray" />
-        </visual>
-    </link>
-    <link name="caster_wheel_link">
-        <xacro:sphere_inertia m="0.5" r="${wheel_radius / 2.0}"  o_xyz="0 0 0" o_rpy="0 0 0" />
-        <collision>
-            <origin xyz="0 0 0" rpy="0 0 0" />
-            <geometry>
-                <sphere radius="${wheel_radius / 2.0}" />
-            </geometry>
-        </collision>
-        <visual>
-            <geometry>
-                <sphere radius="${wheel_radius / 2.0}" />
-            </geometry>
-            <origin xyz="0 0 0" rpy="0 0 0 " />
-            <material name="gray" />
-        </visual>
-    </link>
-    <link name="base_footprint" />
-    <joint name="base_camera_joint" type="fixed">
-        <parent link="base_link" />
-        <child link="camera_link" />
-        <origin xyz="${base_length / 2} 0 ${base_height}" rpy="0 0 0" />
-    </joint>
-    <joint name="base_shoulder_joint" type="revolute">
-        <parent link="base_link" />
-        <child link="shoulder_link" />
-        <origin xyz="0 0 ${base_height}" rpy="0 0 0" />
-        <axis xyz="0 0 1" />
-        <limit lower="${-pi}" upper="${pi}" velocity="100" effort="100" />
-    </joint>
-    <joint name="base_right_wheel_joint" type="continuous">
-        <parent link="base_link" />
-        <child link="right_wheel_link" />
-        <origin xyz="${-base_length / 4.0} ${-(base_width + wheel_length) /
-            2.0} 0" rpy="0 0 0" />
-        <axis xyz="0 1 0" />
-    </joint>
-    <joint name="base_left_wheel_joint" type="continuous">
-        <parent link="base_link" />
-        <child link="left_wheel_link" />
-        <origin xyz="${-base_length / 4.0} ${(base_width + wheel_length) /
-            2.0} 0" rpy="0 0 0" />
-        <axis xyz="0 1 0" />
-    </joint>
-    <joint name="base_caster_wheel_joint" type="fixed">
-        <parent link="base_link" />
-        <child link="caster_wheel_link" />
-        <origin xyz="0.2 0 ${-wheel_radius / 2.0}" rpy="0 0 0" />
-    </joint>
-    <joint name="base_joint" type="fixed">
-        <parent link="base_footprint" />
-        <child link="base_link" />
-        <origin xyz="0 0 ${wheel_radius}" rpy="0 0 0" />
-    </joint>
-</robot>
+/home/fizzer/my_robot_ws/src/my_robot_description/urdf/my_robot.urdf.xacro

File: src/my_robot_description/urdf/my_robot.urdf.xacro (robot description, xacro)
@@ -1,10 +1,10 @@
 <?xml version="1.0"?>
 <robot name="my_robot" xmlns:xacro="http://www.ros.org/wiki/xacro">
-    <xacro:property name="base_length" value="0.6" />
-    <xacro:property name="base_width" value="0.4" />
-    <xacro:property name="base_height" value="0.2" />
-    <xacro:property name="wheel_radius" value="0.1" />
-    <xacro:property name="wheel_length" value="0.05" />
-    <xacro:property name="camera_side_length" value="0.04" />
+    <xacro:property name="base_length" value="0.2" />
+    <xacro:property name="base_width" value="0.15" />
+    <xacro:property name="base_height" value="0.05" />
+    <xacro:property name="wheel_radius" value="0.04" />
+    <xacro:property name="wheel_length" value="0.03" />
+    <xacro:property name="camera_side_length" value="0.03" />
     <xacro:include filename="$(find my_robot_description)/urdf/common_properties.xacro" />
     <xacro:include filename="$(find my_robot_description)/urdf/mobile_base_gazebo.xacro" />
@@ -41,15 +41,4 @@
             <origin xyz="0 0 ${base_height / 2.0}" rpy="0 0 0" />
             <material name="green" />
-        </visual>
-    </link>
-    <link name="shoulder_link">
-        <xacro:cylinder_inertia m="1.0" r="0.1" l="0.3"
-        o_xyz="0 0 0.15" o_rpy="0 0 0" />
-        <visual>
-            <geometry>
-                <cylinder radius="0.1" length="0.3" />
-            </geometry>
-            <origin xyz="0 0 0.15" rpy="0 0 0" />
-            <material name="gray" />
         </visual>
     </link>
@@ -110,11 +99,4 @@
         <origin xyz="${base_length / 2} 0 ${base_height}" rpy="0 0 0" />
     </joint>
-    <joint name="base_shoulder_joint" type="revolute">
-        <parent link="base_link" />
-        <child link="shoulder_link" />
-        <origin xyz="0 0 ${base_height}" rpy="0 0 0" />
-        <axis xyz="0 0 1" />
-        <limit lower="${-pi}" upper="${pi}" velocity="100" effort="100" />
-    </joint>
     <joint name="base_right_wheel_joint" type="continuous">
         <parent link="base_link" />
@@ -134,5 +116,5 @@
         <parent link="base_link" />
         <child link="caster_wheel_link" />
-        <origin xyz="0.2 0 ${-wheel_radius / 2.0}" rpy="0 0 0" />
+        <origin xyz="${base_length / 3.0} 0 ${-wheel_radius / 2.0}" rpy="0 0 0" />
     </joint>
     <joint name="base_joint" type="fixed">

Commit message: FINALLY GOT NPC WORKING

File: install/my_robot_description/share/my_robot_description/urdf/common_properties.xacro (robot description, xacro)
@@ -1 +1,33 @@
-/home/fizzer/my_robot_ws/src/my_robot_description/urdf/common_properties.xacro
+<?xml version="1.0"?>
+<robot xmlns:xacro="http://www.ros.org/wiki/xacro">
+    <!-- Box Inertia Macro -->
+    <xacro:macro name="box_inertia" params="m x y z o_xyz o_rpy">
+    <inertial>
+        <mass value="${m}" />
+        <origin xyz="${o_xyz}" rpy="${o_rpy}" />
+        <inertia ixx="${(m/12) * (y*y + z*z)}" ixy="0" ixz="0"
+                iyy="${(m/12) * (x*x + z*z)}" iyz="0"
+                izz="${(m/12) * (x*x + y*y)}" />
+    </inertial>
+    </xacro:macro>
+    <!-- Cylinder Inertia Macro -->
+    <xacro:macro name="cylinder_inertia" params="m r l o_xyz o_rpy">
+    <inertial>
+        <mass value="${m}" />
+        <origin xyz="${o_xyz}" rpy="${o_rpy}" />
+        <inertia ixx="${(m/12) * (3*r*r + l*l)}" ixy="0" ixz="0"
+                iyy="${(m/12) * (3*r*r + l*l)}" iyz="0"
+                izz="${(m/2) * (r*r)}" />
+    </inertial>
+    </xacro:macro>
+    <!-- Sphere Inertia Macro -->
+    <xacro:macro name="sphere_inertia" params="m r o_xyz o_rpy">
+    <inertial>
+        <mass value="${m}" />
+        <origin xyz="${o_xyz}" rpy="${o_rpy}" />
+        <inertia ixx="${(2/5) * m * r * r}" ixy="0" ixz="0"
+                iyy="${(2/5) * m * r * r}" iyz="0"
+                izz="${(2/5) * m * r * r}" />
+    </inertial>
+    </xacro:macro>
+</robot>

File: install/my_robot_description/share/my_robot_description/urdf/mobile_base_gazebo.xacro (robot description, xacro)
@@ -1 +1,44 @@
-/home/fizzer/my_robot_ws/src/my_robot_description/urdf/mobile_base_gazebo.xacro
+<?xml version="1.0"?>
+<robot xmlns:xacro="http://www.ros.org/wiki/xacro">
+    <xacro:property name="FOV" value="60" />
+    <gazebo>
+        <plugin filename="gz-sim-diff-drive-system" name="gz::sim::systems::DiffDrive">
+            <left_joint>base_left_wheel_joint</left_joint>
+            <right_joint>base_right_wheel_joint</right_joint>
+            <frame_id>odom</frame_id>
+            <child_frame_id>base_footprint</child_frame_id>
+            <wheel_separation>0.45</wheel_separation>
+            <wheel_radius>0.1</wheel_radius>
+        </plugin>
+    </gazebo>
+    <gazebo reference="caster_wheel_link">
+        <mu1 value="0.1" />
+        <mu2 value="0.1" />
+    </gazebo>
+    <gazebo>
+        <plugin
+            filename="gz-sim-joint-state-publisher-system"
+            name="gz::sim::systems::JointStatePublisher">
+        </plugin>
+    </gazebo>
+    <gazebo reference="camera_link">
+        <sensor type="camera" name="drive_camera">
+            <pose relative_to='camera_link'>0 0 0 0 0 0</pose>
+            <camera>
+                <horizontal_fov>${FOV * pi / 180}</horizontal_fov>
+                <image>
+                <width>720</width>
+                <height>480</height>
+                </image>
+                <clip>
+                <near>0.1</near>
+                <far>100</far>
+                </clip>
+            </camera>
+            <always_on>1</always_on>
+            <update_rate>15</update_rate>
+            <visualize>true</visualize>
+            <topic>camera/image_raw</topic>
+        </sensor>
+    </gazebo>
+</robot>

File: install/my_robot_description/share/my_robot_description/urdf/my_robot.urdf.xacro (robot description, xacro)
@@ -1 +1,125 @@
-/home/fizzer/my_robot_ws/src/my_robot_description/urdf/my_robot.urdf.xacro
+<?xml version="1.0"?>
+<robot name="my_robot" xmlns:xacro="http://www.ros.org/wiki/xacro">
+    <xacro:property name="base_length" value="0.2" />
+    <xacro:property name="base_width" value="0.15" />
+    <xacro:property name="base_height" value="0.05" />
+    <xacro:property name="wheel_radius" value="0.04" />
+    <xacro:property name="wheel_length" value="0.03" />
+    <xacro:property name="camera_side_length" value="0.03" />
+    <xacro:include filename="$(find my_robot_description)/urdf/common_properties.xacro" />
+    <xacro:include filename="$(find my_robot_description)/urdf/mobile_base_gazebo.xacro" />
+    <material name="green">
+        <color rgba="0 0.6 0 1" />
+    </material>
+    <material name="gray">
+        <color rgba="0.7 0.7 0.7 1" />
+    </material>
+    <link name="camera_link">
+        <xacro:box_inertia m="0.01" x="${camera_side_length}" y="${camera_side_length}"
+        z="${camera_side_length}" o_xyz="${camera_side_length / 2} 0 0" o_rpy="0 0 0" />
+        <visual>
+            <geometry>
+                <box size="${camera_side_length} ${camera_side_length} ${camera_side_length}" />
+            </geometry>
+            <origin xyz="${camera_side_length / 2} 0 0" rpy="0 0 0" />
+            <material name="gray" />
+        </visual>
+    </link>
+    <link name="base_link">
+        <xacro:box_inertia m="5.0" x="${base_length}" y="${base_width}" z="${base_height}"
+        o_xyz="0 0 ${base_height / 2.0}" o_rpy="0 0 0" />
+        <collision>
+            <origin xyz="0 0 ${base_height / 2.0}" rpy="0 0 0" />
+            <geometry>
+                <box size="${base_length} ${base_width} ${base_height}" />
+            </geometry>
+        </collision>
+        <visual>
+            <geometry>
+                <box size="${base_length} ${base_width} ${base_height}" />
+            </geometry>
+            <origin xyz="0 0 ${base_height / 2.0}" rpy="0 0 0" />
+            <material name="green" />
+        </visual>
+    </link>
+    <link name="right_wheel_link">
+        <xacro:cylinder_inertia m="1.0" r="${wheel_radius}" l="${wheel_length}"
+        o_xyz="0 0 0" o_rpy="${pi / 2.0} 0 0" />
+        <collision>
+            <origin xyz="0 0 0" rpy="0 0 0" />
+            <geometry>
+                <sphere radius="${wheel_radius}" />
+            </geometry>
+        </collision>
+        <visual>
+            <geometry>
+                <cylinder radius="${wheel_radius}" length="${wheel_length}" />
+            </geometry>
+            <origin xyz="0 0 0" rpy="${pi / 2.0} 0 0" />
+            <material name="gray" />
+        </visual>
+    </link>
+    <link name="left_wheel_link">
+        <xacro:cylinder_inertia m="1.0" r="${wheel_radius}" l="${wheel_length}"
+        o_xyz="0 0 0" o_rpy="${pi / 2.0} 0 0" />
+        <collision>
+            <origin xyz="0 0 0" rpy="0 0 0" />
+            <geometry>
+                <sphere radius="${wheel_radius}" />
+            </geometry>
+        </collision>
+        <visual>
+            <geometry>
+                <cylinder radius="${wheel_radius}" length="${wheel_length}" />
+            </geometry>
+            <origin xyz="0 0 0" rpy="${-pi / 2.0} 0 0" />
+            <material name="gray" />
+        </visual>
+    </link>
+    <link name="caster_wheel_link">
+        <xacro:sphere_inertia m="0.5" r="${wheel_radius / 2.0}"  o_xyz="0 0 0" o_rpy="0 0 0" />
+        <collision>
+            <origin xyz="0 0 0" rpy="0 0 0" />
+            <geometry>
+                <sphere radius="${wheel_radius / 2.0}" />
+            </geometry>
+        </collision>
+        <visual>
+            <geometry>
+                <sphere radius="${wheel_radius / 2.0}" />
+            </geometry>
+            <origin xyz="0 0 0" rpy="0 0 0 " />
+            <material name="gray" />
+        </visual>
+    </link>
+    <link name="base_footprint" />
+    <joint name="base_camera_joint" type="fixed">
+        <parent link="base_link" />
+        <child link="camera_link" />
+        <origin xyz="${base_length / 2} 0 ${base_height}" rpy="0 0 0" />
+    </joint>
+    <joint name="base_right_wheel_joint" type="continuous">
+        <parent link="base_link" />
+        <child link="right_wheel_link" />
+        <origin xyz="${-base_length / 4.0} ${-(base_width + wheel_length) /
+            2.0} 0" rpy="0 0 0" />
+        <axis xyz="0 1 0" />
+    </joint>
+    <joint name="base_left_wheel_joint" type="continuous">
+        <parent link="base_link" />
+        <child link="left_wheel_link" />
+        <origin xyz="${-base_length / 4.0} ${(base_width + wheel_length) /
+            2.0} 0" rpy="0 0 0" />
+        <axis xyz="0 1 0" />
+    </joint>
+    <joint name="base_caster_wheel_joint" type="fixed">
+        <parent link="base_link" />
+        <child link="caster_wheel_link" />
+        <origin xyz="${base_length / 3.0} 0 ${-wheel_radius / 2.0}" rpy="0 0 0" />
+    </joint>
+    <joint name="base_joint" type="fixed">
+        <parent link="base_footprint" />
+        <child link="base_link" />
+        <origin xyz="0 0 ${wheel_radius}" rpy="0 0 0" />
+    </joint>
+</robot>
