Commit message: Teleop twist working

File: install/my_robot_description/share/my_robot_description/urdf/my_robot.urdf.xacro (robot description, xacro)
@@ -6,4 +6,6 @@
     <xacro:property name="wheel_radius" value="0.1" />
     <xacro:property name="wheel_length" value="0.05" />
+    <xacro:include filename="$(find my_robot_description)/urdf/common_properties.xacro" />
+    <xacro:include filename="$(find my_robot_description)/urdf/mobile_base_gazebo.xacro" />
     <material name="green">
         <color rgba="0 0.6 0 1" />
@@ -13,4 +15,12 @@
     </material>
     <link name="base_link">
+        <xacro:box_inertia m="5.0" x="${base_length}" y="${base_width}" z="${base_height}"
+        o_xyz="0 0 ${base_height / 2.0}" o_rpy="0 0 0" />
+        <collision>
+            <origin xyz="0 0 ${base_height / 2.0}" rpy="0 0 0" />
+            <geometry>
+                <box size="${base_length} ${base_width} ${base_height}" />
+            </geometry>
+        </collision>
         <visual>
             <geometry>
@@ -22,4 +32,6 @@
     </link>
     <link name="shoulder_link">
+        <xacro:cylinder_inertia m="1.0" r="0.1" l="0.3"
+        o_xyz="0 0 0.15" o_rpy="0 0 0" />
         <visual>
             <geometry>
@@ -31,4 +43,12 @@
     </link>
     <link name="right_wheel_link">
+        <xacro:cylinder_inertia m="1.0" r="${wheel_radius}" l="${wheel_length}"
+        o_xyz="0 0 0" o_rpy="${pi / 2.0} 0 0" />
+        <collision>
+            <origin xyz="0 0 0" rpy="0 0 0" />
+            <geometry>
+                <sphere radius="${wheel_radius}" />
+            </geometry>
+        </collision>
         <visual>
             <geometry>
@@ -40,4 +60,12 @@
     </link>
     <link name="left_wheel_link">
+        <xacro:cylinder_inertia m="1.0" r="${wheel_radius}" l="${wheel_length}"
+        o_xyz="0 0 0" o_rpy="${pi / 2.0} 0 0" />
+        <collision>
+            <origin xyz="0 0 0" rpy="0 0 0" />
+            <geometry>
+                <sphere radius="${wheel_radius}" />
+            </geometry>
+        </collision>
         <visual>
             <geometry>
@@ -49,4 +77,11 @@
     </link>
     <link name="caster_wheel_link">
+        <xacro:sphere_inertia m="0.5" r="${wheel_radius / 2.0}"  o_xyz="0 0 0" o_rpy="0 0 0" />
+        <collision>
+            <origin xyz="0 0 0" rpy="0 0 0" />
+            <geometry>
+                <sphere radius="${wheel_radius / 2.0}" />
+            </geometry>
+        </collision>
         <visual>
             <geometry>

Commit message: all NPCs

File: install/my_robot_description/share/my_robot_description/urdf/my_robot.urdf.xacro (robot description, xacro)
@@ -1,125 +1 @@
-<?xml version="1.0"?>
-<robot name="my_robot" xmlns:xacro="http://www.ros.org/wiki/xacro">
-    <xacro:property name="base_length" value="0.2" />
-    <xacro:property name="base_width" value="0.15" />
-    <xacro:property name="base_height" value="0.05" />
-    <xacro:property name="wheel_radius" value="0.04" />
-    <xacro:property name="wheel_length" value="0.03" />
-    <xacro:property name="camera_side_length" value="0.03" />
-    <xacro:include filename="$(find my_robot_description)/urdf/common_properties.xacro" />
-    <xacro:include filename="$(find my_robot_description)/urdf/mobile_base_gazebo.xacro" />
-    <material name="green">
-        <color rgba="0 0.6 0 1" />
-    </material>
-    <material name="gray">
-        <color rgba="0.7 0.7 0.7 1" />
-    </material>
-    <link name="camera_link">
-        <xacro:box_inertia m="0.01" x="${camera_side_length}" y="${camera_side_length}"
-        z="${camera_side_length}" o_xyz="${camera_side_length / 2} 0 0" o_rpy="0 0 0" />
-        <visual>
-            <geometry>
-                <box size="${camera_side_length} ${camera_side_length} ${camera_side_length}" />
-            </geometry>
-            <origin xyz="${camera_side_length / 2} 0 0" rpy="0 0 0" />
-            <material name="gray" />
-        </visual>
-    </link>
-    <link name="base_link">
-        <xacro:box_inertia m="5.0" x="${base_length}" y="${base_width}" z="${base_height}"
-        o_xyz="0 0 ${base_height / 2.0}" o_rpy="0 0 0" />
-        <collision>
-            <origin xyz="0 0 ${base_height / 2.0}" rpy="0 0 0" />
-            <geometry>
-                <box size="${base_length} ${base_width} ${base_height}" />
-            </geometry>
-        </collision>
-        <visual>
-            <geometry>
-                <box size="${base_length} ${base_width} ${base_height}" />
-            </geometry>
-            <origin xyz="0 0 ${base_height / 2.0}" rpy="0 0 0" />
-            <material name="green" />
-        </visual>
-    </link>
-    <link name="right_wheel_link">
-        <xacro:cylinder_inertia m="1.0" r="${wheel_radius}" l="${wheel_length}"
-        o_xyz="0 0 0" o_rpy="${pi / 2.0} 0 0" />
-        <collision>
-            <origin xyz="0 0 0" rpy="0 0 0" />
-            <geometry>
-                <sphere radius="${wheel_radius}" />
-            </geometry>
-        </collision>
-        <visual>
-            <geometry>
-                <cylinder radius="${wheel_radius}" length="${wheel_length}" />
-            </geometry>
-            <origin xyz="0 0 0" rpy="${pi / 2.0} 0 0" />
-            <material name="gray" />
-        </visual>
-    </link>
-    <link name="left_wheel_link">
-        <xacro:cylinder_inertia m="1.0" r="${wheel_radius}" l="${wheel_length}"
-        o_xyz="0 0 0" o_rpy="${pi / 2.0} 0 0" />
-        <collision>
-            <origin xyz="0 0 0" rpy="0 0 0" />
-            <geometry>
-                <sphere radius="${wheel_radius}" />
-            </geometry>
-        </collision>
-        <visual>
-            <geometry>
-                <cylinder radius="${wheel_radius}" length="${wheel_length}" />
-            </geometry>
-            <origin xyz="0 0 0" rpy="${-pi / 2.0} 0 0" />
-            <material name="gray" />
-        </visual>
-    </link>
-    <link name="caster_wheel_link">
-        <xacro:sphere_inertia m="0.5" r="${wheel_radius / 2.0}"  o_xyz="0 0 0" o_rpy="0 0 0" />
-        <collision>
-            <origin xyz="0 0 0" rpy="0 0 0" />
-            <geometry>
-                <sphere radius="${wheel_radius / 2.0}" />
-            </geometry>
-        </collision>
-        <visual>
-            <geometry>
-                <sphere radius="${wheel_radius / 2.0}" />
-            </geometry>
-            <origin xyz="0 0 0" rpy="0 0 0 " />
-            <material name="gray" />
-        </visual>
-    </link>
-    <link name="base_footprint" />
-    <joint name="base_camera_joint" type="fixed">
-        <parent link="base_link" />
-        <child link="camera_link" />
-        <origin xyz="${base_length / 2} 0 ${base_height}" rpy="0 0 0" />
-    </joint>
-    <joint name="base_right_wheel_joint" type="continuous">
-        <parent link="base_link" />
-        <child link="right_wheel_link" />
-        <origin xyz="${-base_length / 4.0} ${-(base_width + wheel_length) /
-            2.0} 0" rpy="0 0 0" />
-        <axis xyz="0 1 0" />
-    </joint>
-    <joint name="base_left_wheel_joint" type="continuous">
-        <parent link="base_link" />
-        <child link="left_wheel_link" />
-        <origin xyz="${-base_length / 4.0} ${(base_width + wheel_length) /
-            2.0} 0" rpy="0 0 0" />
-        <axis xyz="0 1 0" />
-    </joint>
-    <joint name="base_caster_wheel_joint" type="fixed">
-        <parent link="base_link" />
-        <child link="caster_wheel_link" />
-        <origin xyz="${base_length / 3.0} 0 ${-wheel_radius / 2.0}" rpy="0 0 0" />
-    </joint>
-    <joint name="base_joint" type="fixed">
-        <parent link="base_footprint" />
-        <child link="base_link" />
-        <origin xyz="0 0 ${wheel_radius}" rpy="0 0 0" />
-    </joint>
-</robot>
+/home/fizzer/my_robot_ws/src/my_robot_description/urdf/my_robot.urdf.xacro

File: src/my_robot_description/urdf/my_robot.urdf.xacro (robot description, xacro)
@@ -123,3 +123,15 @@
         <origin xyz="0 0 ${wheel_radius}" rpy="0 0 0" />
     </joint>
+    <gazebo>
+        <plugin filename="gz-sim-pose-publisher-system"
+            name="gz::sim::systems::PosePublisher">
+            <publish_model_pose>true</publish_model_pose>
+            <publish_link_pose>false</publish_link_pose>
+            <publish_sensor_pose>false</publish_sensor_pose>
+            <publish_collision_pose>false</publish_collision_pose>
+            <publish_visual_pose>false</publish_visual_pose>
+            <update_frequency>50</update_frequency>
+            <use_pose_vector_msg>false</use_pose_vector_msg>
+        </plugin>
+    </gazebo>
 </robot>
